File: hardware/max3421e-rpi-uhat.kicad_pcb (KiCad board)
At the start: 2 copper layers, 0 parts

Commit message: Design version 1.0
Parts:
- added C1: 4.7nF, Capacitor_SMD:C_0603_1608Metric, F.Cu at (119.5, 64.5)
- added C2: 18pF, Capacitor_SMD:C_0603_1608Metric, F.Cu at (87.7, 64.5)
- added C3: 18pF, Capacitor_SMD:C_0603_1608Metric, F.Cu at (84.8, 61.5)
- added C4: 0.1uF, Capacitor_SMD:C_0603_1608Metric, F.Cu at (85.5, 58.5)
- added C5: 0.1uF, Capacitor_SMD:C_0603_1608Metric, F.Cu at (97.5, 59.0)
- added C6: 150uF, Capacitor_SMD:CP_Elec_6.3x5.4, F.Cu at (78.9, 61.5)
- added C7: 0.1uF, Capacitor_SMD:C_0603_1608Metric, F.Cu at (76.7, 54.6)
- added H1: MountingHole, rpiuhat:MountingHole_2.75mm_6.2mm, F.Cu at (70.0, 46.5)
- added H2: MountingHole, rpiuhat:MountingHole_2.75mm_6.2mm, F.Cu at (128.0, 46.5)
- added H3: MountingHole, rpiuhat:MountingHole_2.75mm_6.2mm, F.Cu at (70.0, 69.5)
- added H4: MountingHole, rpiuhat:MountingHole_2.75mm_6.2mm, F.Cu at (128.0, 69.5)
- added J1: Raspberry_Pi_GPIO, Connector_PinSocket_2.54mm:PinSocket_2x20_P2.54mm_Vertical, B.Cu at (74.9, 47.8)
- added J2: USB_A, rpiuhat:USB-A-SMD_FUS270-FSBW5K, F.Cu at (107.9, 61.0)
- added J3: GPIN, Connector_PinHeader_2.54mm:PinHeader_1x07_P2.54mm_Vertical, F.Cu at (80.0, 68.1)
- added J4: GPOUT, Connector_PinHeader_2.54mm:PinHeader_1x07_P2.54mm_Vertical, F.Cu at (118.1, 52.9)
- added R1: 33R, Resistor_SMD:R_0603_1608Metric, F.Cu at (85.5, 56.5)
- added R2: 33R, Resistor_SMD:R_0603_1608Metric, F.Cu at (85.5, 55.0)
- added R3: 1M, Resistor_SMD:R_0603_1608Metric, F.Cu at (119.5, 66.5)
- added R4: 10K, Resistor_SMD:R_0603_1608Metric, F.Cu at (82.3, 55.9)
- added REF**: OSHW-Logo2_9.8x8mm_SilkScreen, Symbol:OSHW-Logo2_9.8x8mm_SilkScreen, B.Cu at (117.8, 64.8)
- added U1: MAX3421EEHJ+T, rpiuhat:QFP50P700X700X120-32N, F.Cu at (92.2, 56.3)
- added U2: TPS2065CDBVR, rpiuhat:SOT95P280X145-5N, F.Cu at (79.5, 55.2)
- added Y1: 12MHz, Crystal:Crystal_SMD_3225-4Pin_3.2x2.5mm, F.Cu at (87.5, 61.5)
Routing:
- net +3V3: track 0.00 -> 57.3 mm, vias 0 -> 2
- net VBUS: track 0.00 -> 31.0 mm, vias 0 -> 2
- net GND: track 0.00 -> 29.0 mm, vias 0 -> 13
- net /D_P: track 0.00 -> 27.7 mm, vias 0 -> 2
- net /D_N: track 0.00 -> 27.4 mm, vias 0 -> 2
- net /GPOUT1: track 0.00 -> 24.0 mm
- net /GPOUT2: track 0.00 -> 21.3 mm
- net /GPOUT3: track 0.00 -> 18.6 mm
- net INT1: track 0.00 -> 18.2 mm
- net /GPIN1: track 0.00 -> 17.8 mm
- net FAULT: track 0.00 -> 17.2 mm, vias 0 -> 2
- net VUSB_EN: track 0.00 -> 16.6 mm, vias 0 -> 2
- net /SS: track 0.00 -> 16.3 mm
- net /GPIN2: track 0.00 -> 15.9 mm
- net /GPOUT4: track 0.00 -> 15.8 mm
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- added copper zone on B.Cu, net GND
- added copper zone on F.Cu, net GND
- added copper zone on F.Cu, net Net-(J2-Shield)
Other:
- board outline added: 65 x 30 mm
- board text added: "GPIN [1 .. 7]"
- board text added: "GPOUT [7 ... 1]"
- board text added: "Raspberry Pi MAX3421E uHAT Version 1.0 (11/23) https://github.com/StarGate01/max3421e-rpi-uhat"
