File: hardware/max3421e-rpi-uhat.kicad_sch (KiCad schematic)
At the start: 1 part, among them U1 MAX3421EEHJ+T

Commit message: Design version 1.0
Parts:
- added C1: 4.7nF, Capacitor_SMD:C_0603_1608Metric, symbol Device:C
- added C2, C3: 18pF, Capacitor_SMD:C_0603_1608Metric, symbol Device:C
- added C4, C5, C7: 0.1uF, Capacitor_SMD:C_0603_1608Metric, symbol Device:C
- added C6: 150uF, Capacitor_SMD:CP_Elec_6.3x5.4, symbol Device:C_Polarized
- added H1, H2, H3, H4: MountingHole, rpiuhat:MountingHole_2.75mm_6.2mm, symbol Mechanical:MountingHole
- added J1: Raspberry_Pi_GPIO, Connector_PinSocket_2.54mm:PinSocket_2x20_P2.54mm_Vertical, symbol Connector:Raspberry_Pi_2_3
- added J2: USB_A, rpiuhat:USB-A-SMD_FUS270-FSBW5K, symbol Connector:USB_A
- added J3: GPIN, Connector_PinHeader_2.54mm:PinHeader_1x07_P2.54mm_Vertical, symbol Connector_Generic:Conn_01x07
- added J4: GPOUT, Connector_PinHeader_2.54mm:PinHeader_1x07_P2.54mm_Vertical, symbol Connector_Generic:Conn_01x07
- added R1, R2: 33R, Resistor_SMD:R_0603_1608Metric, symbol Device:R
- added R3: 1M, Resistor_SMD:R_0603_1608Metric, symbol Device:R
- added R4: 10K, Resistor_SMD:R_0603_1608Metric, symbol Device:R
- added U2: TPS2065CDBVR, rpiuhat:SOT95P280X145-5N, symbol rpiuhat:TPS2051CDBVR
- added Y1: 12MHz, Crystal:Crystal_SMD_3225-4Pin_3.2x2.5mm, symbol Device:Crystal_GND24
- U1: Distributor (none) -> LCSC; Distributor Part (none) -> C2651881; MPN (none) -> MAX3421EEHJ+T; Manufacturer (none) -> Analog Devices Inc./Maxim Integrated
Connections:
- net GPIN7: now reaches U1.1 (GPIN7)
- net GPIN7: now also J3.7 (Pin_7)
- net GPOUT6: now reaches U1.10 (GPOUT6)
- net GPOUT6: now also J4.6 (Pin_6)
- net GPOUT7: now reaches U1.11 (GPOUT7)
- net GPOUT7: now also J4.7 (Pin_7)
- net +3V3: now reaches U1.12 (~{RES})
- net +3V3: now also U1.2 (VL), U1.23 (VCC), C4.1, C5.1, J1.1 (3V3), J1.17 (3V3), R4.2
- net SCLK: now reaches U1.13 (SCLK)
- net SCLK: now also J1.23 (SCLK0/GPIO11)
- net SS: now reaches U1.14 (~{SS})
- net SS: now also J1.24 (~{CE0}/GPIO8)
- net MISO: now reaches U1.15 (MISO)
- net MISO: now also J1.21 (MISO0/GPIO9)
- net MOSI: now reaches U1.16 (MOSI)
- net MOSI: now also J1.19 (MOSI0/GPIO10)
- net INT2: now reaches U1.17 (GPX)
- net INT2: now also J1.18 (GPIO24)
- net INT1: now reaches U1.18 (INT)
- net INT1: now also J1.22 (GPIO25)
- net GND: now reaches U1.19 (GND_2)
- net GND: now also U1.3 (GND_1), C1.1, C2.1, C3.1, C4.2, C5.2, C6.2, C7.2, J1.14 (GND), J1.20 (GND), J1.25 (GND), J1.30 (GND), J1.34 (GND), J1.39 (GND), J1.6 (GND), J1.9 (GND), J2.4 (GND), R3.2, U2.2 (GND), Y1.2, Y1.4
- net at U1.20 (D-): now also R2.1
- net at U1.21 (D+): now also R1.1
- net XTAL_1: now reaches U1.24 (XI)
- net XTAL_1: now also C3.2, Y1.3
- net XTAL_0: now reaches U1.25 (XO)
- net XTAL_0: now also C2.2, Y1.1
- net FAULT: now reaches U1.26 (GPIN0)
- net FAULT: now also R4.1, U2.3 (~{FLT})
- net GPIN1: now reaches U1.27 (GPIN1)
- net GPIN1: now also J3.1 (Pin_1)
- net GPIN2: now reaches U1.28 (GPIN2)
- net GPIN2: now also J3.2 (Pin_2)
- net GPIN3: now reaches U1.29 (GPIN3)
- net GPIN3: now also J3.3 (Pin_3)
- net GPIN4: now reaches U1.30 (GPIN4)
- net GPIN4: now also J3.4 (Pin_4)
- net GPIN5: now reaches U1.31 (GPIN5)
- net GPIN5: now also J3.5 (Pin_5)
- net GPIN6: now reaches U1.32 (GPIN6)
- net GPIN6: now also J3.6 (Pin_6)
- net VUSB_EN: now reaches U1.4 (GPOUT0)
- net VUSB_EN: now also U2.4 (EN/~{EN})
- net GPOUT1: now reaches U1.5 (GPOUT1)
- net GPOUT1: now also J4.1 (Pin_1)
- net GPOUT2: now reaches U1.6 (GPOUT2)
- net GPOUT2: now also J4.2 (Pin_2)
- net GPOUT3: now reaches U1.7 (GPOUT3)
- net GPOUT3: now also J4.3 (Pin_3)
- net GPOUT4: now reaches U1.8 (GPOUT4)
- net GPOUT4: now also J4.4 (Pin_4)
- net GPOUT5: now reaches U1.9 (GPOUT5)
- net GPOUT5: now also J4.5 (Pin_5)
- new net: C1.2, J2.5 (Shield), R3.1
- new net +5V: C7.1, J1.2 (5V), J1.4 (5V), U2.5 (IN)
- new net D_N: J2.2 (D-), R2.2
- new net D_P: J2.3 (D+), R1.2
- new net VBUS: C6.1, J2.1 (VBUS), U2.1 (OUT)
- no-connect marks 0 -> 23
Other:
- note added: "MAX3421E AUX GPIO"
- note added: "MAX3421E CLOCK"
- note added: "RASPBERRY PI INTERFACE"
- note added: "USB OVERCURRENT+CONTROL SWITCH (500mA)"
- note added: "USB-A PORT"
- moved on the sheet: U1
